Commit message: idk how odom work...

File: URDF/roar_bot.urdf.xacro (robot description, xacro)
@@ -10,4 +10,19 @@
   <xacro:property name="iphone_width" value="0.02"/>
   <xacro:property name="iphone_length" value="0.09"/>
+    <!-- Define intertial property macros  -->
+  <xacro:macro name="box_inertia" params="m w h d">
+    <inertial>
+      <origin xyz="0 0 0" rpy="${pi/2} 0 ${pi/2}"/>
+      <mass value="${m}"/>
+      <inertia ixx="${(m/12) * (h*h + d*d)}" ixy="0.0" ixz="0.0" iyy="${(m/12) * (w*w + d*d)}" iyz="0.0" izz="${(m/12) * (w*w + h*h)}"/>
+    </inertial>
+  </xacro:macro>
+  <xacro:macro name="cylinder_inertia" params="m r h">
+    <inertial>
+      <origin xyz="0 0 0" rpy="${pi/2} 0 0" />
+      <mass value="${m}"/>
+      <inertia ixx="${(m/12) * (3*r*r + h*h)}" ixy = "0" ixz = "0" iyy="${(m/12) * (3*r*r + h*h)}" iyz = "0" izz="${(m/2) * (r*r)}"/>
+    </inertial>
+  </xacro:macro>
     <!-- Robot Base -->
   <link name="base_link">
@@ -20,16 +35,29 @@
       </material>
     </visual>
+    <collision>
+        <geometry>
+          <box size="${base_width} ${base_length} ${base_height}"/>
+        </geometry>
+      </collision>
+      <xacro:box_inertia m="15" w="${base_width}" d="${base_length}" h="${base_height}"/>
   </link>
   <!-- iphone mount -->
   <link name="iphone_link">
     <visual>
-      <origin xyz="0 0 0" rpy="0 0 0"/>
-      <geometry>
-        <box size="${iphone_length} ${iphone_width}  ${iphone_height}"/>
-      </geometry>
+        <origin xyz="0 0 0" rpy="0 0 0"/>
+        <geometry>
+          <box size="${iphone_length} ${iphone_width}  ${iphone_height}"/>
+        </geometry>
       <material name="blue">
         <color rgba="0 0 0 1"/>
       </material>
     </visual>
+     <collision>
+        <origin xyz="0 0 0" rpy="0 0 0"/>
+        <geometry>
+          <box size="${iphone_length} ${iphone_width}  ${iphone_height}"/>
+        </geometry>
+      </collision>
+      <xacro:box_inertia m="5" w="${iphone_width}" d="${iphone_length}" h="${iphone_height}"/>
   </link>
   <joint name="$iphone" type="fixed">
@@ -42,8 +70,8 @@
     <link name="${prefix}_link">
       <visual>
-        <origin xyz="0 0 0" rpy="0 ${pi/2} 0"/>
-        <geometry>
-            <cylinder radius="${wheel_radius}" length="${wheel_width}"/>
-        </geometry>
+            <origin xyz="0 0 0" rpy="0 ${pi/2} 0"/>
+            <geometry>
+                <cylinder radius="${wheel_radius}" length="${wheel_width}"/>
+            </geometry>
         <material name="Gray">
           <color rgba="0.5 0.5 0.5 1.0"/>
@@ -51,4 +79,11 @@
       </visual>
     </link>
+    <collision>
+      <origin xyz="0 0 0" rpy="0 ${pi/2} 0"/>
+      <geometry>
+          <cylinder radius="${wheel_radius}" length="${wheel_width}"/>
+      </geometry>
+    </collision>
+    <xacro:cylinder_inertia m="0.5" r="${wheel_radius}" h="${wheel_width}"/>
     <joint name="${prefix}_joint" type="continuous">
       <parent link="base_link"/>

Commit message: now it spins correctly, but im pretty sure the naming is wrong

File: URDF/roar_bot.urdf.xacro (robot description, xacro)
@@ -42,4 +42,12 @@
       <xacro:box_inertia m="15" w="${base_width}" d="${base_length}" h="${base_height}"/>
   </link>
+  <!-- Robot Footprint -->
+  <!-- Robot Footprint -->
+  <link name="base_footprint"/>
+  <joint name="base_joint" type="fixed">
+    <parent link="base_link"/>
+    <child link="base_footprint"/>
+    <origin xyz="0.0 0.0 0.0" rpy="0 0 0"/>
+  </joint>
   <!-- iphone mount -->
   <link name="iphone_link">
@@ -61,5 +69,5 @@
       <xacro:box_inertia m="5" w="${iphone_width}" d="${iphone_length}" h="${iphone_height}"/>
   </link>
-  <joint name="$iphone" type="fixed">
+  <joint name="iphone" type="fixed">
       <parent link="base_link"/>
       <child link="iphone_link"/>
